Commit message: add pr2 dual arm urdf

File: python/pybullet/grasping_demo/pr2_description/urdf/pr2_lgripper.urdf (robot description, URDF)
Before this commit: robot pr2, 11 links, 10 joints
Links:
- removed link l_gripper_l_finger_tip_frame
- added link pseudo_slider2_link
- added link pseudo_slider_link
- added link pseudo_yrot_link
Joints:
- removed joint l_gripper_joint
- added joint xslide: type prismatic, parent pseudo_slider_link, child pseudo_slider2_link, origin xyz=0.0 0.0 0, axis 0 1 0, limit lower=-15 upper=15 effort=1000.0 velocity=5
- added joint yrot: type continuous, parent pseudo_yrot_link, child l_gripper_palm_link, origin xyz=0.0 0.0 0, axis 0 1 0
- added joint zslide: type prismatic, parent pseudo_slider2_link, child pseudo_yrot_link, origin xyz=0.0 0.0 0, axis 1 0 0, limit lower=-15 upper=15 effort=1000.0 velocity=5

File: python/pybullet/grasping_demo/pr2_description/urdf/pr2_rgripper.urdf (robot description, URDF)
Before this commit: robot pr2, 11 links, 10 joints
Links:
- removed link r_gripper_l_finger_tip_frame
- added link pseudo_slider2_link
- added link pseudo_slider_link
- added link pseudo_yrot_link
Joints:
- removed joint r_gripper_joint
- added joint xslide: type prismatic, parent pseudo_slider_link, child pseudo_slider2_link, origin xyz=0.0 0.0 0, axis 0 1 0, limit lower=-15 upper=15 effort=1000.0 velocity=5
- added joint yrot: type continuous, parent pseudo_yrot_link, child r_gripper_palm_link, origin xyz=0.0 0.0 0, axis 0 1 0
- added joint zslide: type prismatic, parent pseudo_slider2_link, child pseudo_yrot_link, origin xyz=0.0 0.0 0, axis 1 0 0, limit lower=-15 upper=15 effort=1000.0 velocity=5
